Commit message: feat: added robot bringup skeleton + description

File: src/robot_description/urdf/my_amr.urdf.xacro (robot description, xacro)
@@ -1,4 +1,5 @@
 <?xml version="1.0"?>
 <robot name="my_amr" xmlns:xacro="http://www.ros.org/wiki/xacro">
+  <!-- Mesh scale: adjust if your STLs were exported in mm instead of meters -->
   <xacro:property name="mesh_scale" value="0.001 0.001 0.001"/>
   <!-- ======================== Base ======================== -->
@@ -11,11 +12,14 @@
   <link name="base_link">
     <visual>
+      <origin rpy="0 0 0.0"/>
       <geometry>
-        <mesh filename="package://robot_description/meshes/body.stl" scale="${mesh_scale}"/>
+        <mesh filename="package://robot_description/meshes/body_ccw_90.stl" scale="${mesh_scale}"/>
       </geometry>
+      <material name="blue"><color rgba="0.2 0.4 0.8 1"/></material>
     </visual>
     <collision>
+      <origin rpy="0 0 0.0"/>
       <geometry>
-        <mesh filename="package://robot_description/meshes/body.stl" scale="${mesh_scale}"/>
+        <mesh filename="package://robot_description/meshes/body_ccw_90.stl" scale="${mesh_scale}"/>
       </geometry>
     </collision>
@@ -29,17 +33,20 @@
     <parent link="base_link"/>
     <child link="left_wheel"/>
-    <origin xyz="0.230 0.0 0.0" rpy="-1.5708 0 0"/>
-    <axis xyz="1 0 0"/>
+    <origin xyz="0.0 0.230 0.0" rpy="1.5708 0 0"/>
+    <axis xyz="0 0 1"/>
   </joint>
   <link name="left_wheel">
     <visual>
+      <origin rpy="0 0 0"/>
       <geometry>
-        <mesh filename="package://robot_description/meshes/wheel.stl" scale="${mesh_scale}"/>
+        <mesh filename="package://robot_description/meshes/wheel_y_ccw_90.stl" scale="${mesh_scale}"/>
       </geometry>
+      <material name="dark"><color rgba="0.1 0.1 0.1 1"/></material>
     </visual>
     <collision>
+      <origin rpy="0 0 0"/>
       <geometry>
-        <mesh filename="package://robot_description/meshes/wheel.stl" scale="${mesh_scale}"/>
-      </geometry>
+          <mesh filename="package://robot_description/meshes/wheel_y_ccw_90.stl" scale="${mesh_scale}"/>
+        </geometry>
     </collision>
     <inertial>
@@ -51,18 +58,20 @@
     <parent link="base_link"/>
     <child link="right_wheel"/>
-    <origin xyz="-0.230 0.0 0.0" rpy="1.5708 0 0"/>
-    <axis xyz="1 0 0"/>
+    <origin xyz="0.0 -0.230 0.0" rpy="-1.5708 0 0"/>
+    <axis xyz="0 0 1"/>
   </joint>
   <link name="right_wheel">
     <visual>
-      <origin rpy="0 3.14159 0"/>
+      <!-- rpy="0 3.14159 0" flips the mesh if the right side appears mirrored -->
+      <origin rpy="0 0 0"/>
       <geometry>
-        <mesh filename="package://robot_description/meshes/wheel.stl" scale="${mesh_scale}"/>
+        <mesh filename="package://robot_description/meshes/wheel_y_ccw_90.stl" scale="${mesh_scale}"/>
       </geometry>
+      <material name="dark"><color rgba="0.1 0.1 0.1 1"/></material>
     </visual>
     <collision>
       <geometry>
-        <mesh filename="package://robot_description/meshes/wheel.stl" scale="${mesh_scale}"/>
-      </geometry>
+          <mesh filename="package://robot_description/meshes/wheel_y_ccw_90.stl" scale="${mesh_scale}"/>
+        </geometry>
     </collision>
     <inertial>
@@ -75,7 +84,14 @@
     <parent link="base_link"/>
     <child link="front_left_caster"/>
-    <origin xyz="0.210 0.335 -0.031"/>
+    <origin xyz=" 0.335 0.210 -0.031"/>
   </joint>
   <link name="front_left_caster">
+    <visual>
+      <geometry><sphere radius="0.05"/></geometry>
+      <material name="dark"><color rgba="0.1 0.1 0.1 1"/></material>
+    </visual>
+    <collision>
+      <geometry><sphere radius="0.05"/></geometry>
+    </collision>
     <inertial>
       <mass value="0.1"/>
@@ -86,7 +102,14 @@
     <parent link="base_link"/>
     <child link="rear_left_caster"/>
-    <origin xyz="-0.210 0.335 -0.031"/>
+    <origin xyz="0.335 -0.210 -0.031"/>
   </joint>
   <link name="rear_left_caster">
+    <visual>
+      <geometry><sphere radius="0.05"/></geometry>
+      <material name="dark"><color rgba="0.1 0.1 0.1 1"/></material>
+    </visual>
+    <collision>
+      <geometry><sphere radius="0.05"/></geometry>
+    </collision>
     <inertial>
       <mass value="0.1"/>
@@ -97,7 +120,14 @@
     <parent link="base_link"/>
     <child link="front_right_caster"/>
-    <origin xyz="0.210 -0.335 -0.031"/>
+    <origin xyz="-0.335 0.210 -0.031"/>
   </joint>
   <link name="front_right_caster">
+    <visual>
+      <geometry><sphere radius="0.05"/></geometry>
+      <material name="dark"><color rgba="0.1 0.1 0.1 1"/></material>
+    </visual>
+    <collision>
+      <geometry><sphere radius="0.05"/></geometry>
+    </collision>
     <inertial>
       <mass value="0.1"/>
@@ -108,7 +138,14 @@
     <parent link="base_link"/>
     <child link="rear_right_caster"/>
-    <origin xyz="-0.210 -0.335 -0.031"/>
+    <origin xyz="-0.335 -0.210 -0.031"/>
   </joint>
   <link name="rear_right_caster">
+    <visual>
+      <geometry><sphere radius="0.05"/></geometry>
+      <material name="dark"><color rgba="0.1 0.1 0.1 1"/></material>
+    </visual>
+    <collision>
+      <geometry><sphere radius="0.05"/></geometry>
+    </collision>
     <inertial>
       <mass value="0.1"/>
@@ -120,12 +157,15 @@
     <parent link="base_link"/>
     <child link="lidar_link"/>
-    <origin xyz="0.0 -0.400 0.110"/>
+    <!-- lidar body mount: mount height (0.08) + sensor height (0.039) -->
+    <origin xyz="0.400 0 0.110"/>
   </joint>
   <link name="lidar_link">
     <visual>
+      <!-- mesh Z starts at 0 (sensor base); shift down so it renders below the scan frame -->
       <origin xyz="0 0 -0.030"/>
       <geometry>
-        <mesh filename="package://robot_description/meshes/rplidar_s2.stl" scale="${mesh_scale}"/>
+        <mesh filename="package://robot_description/meshes/rplidar_s2_frame_aligned.stl" scale="${mesh_scale}"/>
       </geometry>
+      <material name="dark"><color rgba="0.1 0.1 0.1 1"/></material>
     </visual>
     <inertial>
@@ -143,6 +183,7 @@
     <visual>
       <geometry>
-        <mesh filename="package://robot_description/meshes/ellipse_micro_ahrs.stl" scale="${mesh_scale}"/>
+        <mesh filename="package://robot_description/meshes/ellipse_micro_ahrs_ccw_90.stl" scale="${mesh_scale}"/>
       </geometry>
+      <material name="dark"><color rgba="0.1 0.1 0.1 1"/></material>
     </visual>
     <inertial>

Commit message: feat: added teleoperation layer and configured main vel pipeline

File: src/robot_description/urdf/my_amr.urdf.xacro (robot description, xacro)
@@ -34,5 +34,6 @@
     <child link="left_wheel"/>
     <origin xyz="0.0 0.230 0.0" rpy="1.5708 0 0"/>
-    <axis xyz="0 0 1"/>
+    <!-- Match the right wheel's rotation direction in the base frame. -->
+    <axis xyz="0 0 -1"/>
   </joint>
   <link name="left_wheel">

Commit message: feat: added lidar dock detection prototype

File: src/robot_description/urdf/my_amr.urdf.xacro (robot description, xacro)
@@ -33,5 +33,5 @@
     <parent link="base_link"/>
     <child link="left_wheel"/>
-    <origin xyz="0.0 0.230 0.0" rpy="1.5708 0 0"/>
+    <origin xyz="0.0 0.274 0.0" rpy="1.5708 0 0"/>
     <!-- Match the right wheel's rotation direction in the base frame. -->
     <axis xyz="0 0 -1"/>
@@ -59,5 +59,5 @@
     <parent link="base_link"/>
     <child link="right_wheel"/>
-    <origin xyz="0.0 -0.230 0.0" rpy="-1.5708 0 0"/>
+    <origin xyz="0.0 -0.274 0.0" rpy="-1.5708 0 0"/>
     <axis xyz="0 0 1"/>
   </joint>
